Commit message: corrected tf_broadcaster

File: src/robot_description/urdf/robot.xacro (robot description, xacro)
@@ -9,5 +9,5 @@
 	<xacro:property name="base_Ix" value="${base_mass*(base_hight*base_hight+base_width*base_width)/12}"/>
 	<xacro:property name="base_Iy" value="${base_mass*(base_length*base_length+base_hight*base_hight)/12}"/>
-	<xacro:property name="base_Iz" value="${base_mass*(base_length*base_length+base_width*base_width)/12}"/>
+	<xacro:property name="base_Iz" value="${base_mass*(base_length*base_length+base_width*base_width)/12 * 0.5}"/>
 	<xacro:property name="wheel_radius" value="0.1"/>
 	<xacro:property name="wheel_length" value="0.1"/>
@@ -60,6 +60,6 @@
 		</link>
 		<gazebo reference="{prefix}_wheel">
-			<mu1 value="10"/>
-			<mu2 value="0.5"/>
+			<mu1 value="0.8"/>
+			<mu2 value="0.8"/>
 			<fdir value="1 0 0"/>
 			<material>Gazebo/Black</material>
@@ -78,4 +78,20 @@
 	<xacro:wheel prefix="left_front" xyz_offsets="${base_length/2} -${(base_width+wheel_length)/2} -${base_hight/4}"/>
 	<xacro:wheel prefix="left_rear" xyz_offsets="-${base_length/2} -${(base_width+wheel_length)/2} -${base_hight/4}"/>
+	<gazebo reference="base_link">
+		<material>Gazebo/Blue</material>
+	</gazebo>
+	<gazebo reference="right_front_wheel">
+		<material>Gazebo/Black</material>
+	</gazebo>
+	<gazebo reference="right_rear_wheel">
+		<material>Gazebo/Black</material>
+	</gazebo>
+	<gazebo reference="left_front_wheel">
+		<material>Gazebo/Black</material>
+	</gazebo>
+	<gazebo reference="left_rear_wheel">
+		<material>Gazebo/Black</material>
+	</gazebo>
+	<!-- Hokuyo Laser -->
 	<joint name="hokuyo_joint" type="fixed">
 		<origin xyz="${base_length/2 - base_length/4} 0 ${base_hight/2 + 0.05}" rpy="0 0 0"/>
@@ -83,5 +99,4 @@
 		<child link="hokuyo_link"/>
 	</joint>
-	<!-- Hokuyo Laser -->
 	<link name="hokuyo_link">
 		<collision>
@@ -100,19 +115,4 @@
 		</inertial>
 	</link>
-	<gazebo reference="base_link">
-		<material>Gazebo/Blue</material>
-	</gazebo>
-	<gazebo reference="right_front_wheel">
-		<material>Gazebo/Black</material>
-	</gazebo>
-	<gazebo reference="right_rear_wheel">
-		<material>Gazebo/Black</material>
-	</gazebo>
-	<gazebo reference="left_front_wheel">
-		<material>Gazebo/Black</material>
-	</gazebo>
-	<gazebo reference="left_rear_wheel">
-		<material>Gazebo/Black</material>
-	</gazebo>
 	<gazebo reference="hokuyo_link">
 		<sensor name="head_hokuyo_sensor" type="gpu_ray">
@@ -140,5 +140,5 @@
 			</ray>
 			<plugin filename="libgazebo_ros_gpu_laser.so" name="gazebo_ros_head_hokuyo_controller">
-				<topicName>/robot/laser/scan</topicName>
+				<topicName>/gazebo/laser_scan</topicName>
 				<frameName>hokuyo_link</frameName>
 			</plugin>

Commit message: added IMU

File: src/robot_description/urdf/robot.xacro (robot description, xacro)
@@ -15,4 +15,12 @@
 	<xacro:property name="wheel_Iz" value="${wheel_mass*wheel_radius*wheel_radius/2}"/>
 	<xacro:property name="wheel_Ix" value="${wheel_mass*(3*wheel_radius*wheel_radius+wheel_length*wheel_length)/12}"/>
+	<joint name="base_footprint_joint" type="fixed">
+    	<axis xyz="0 0 0"/>
+    	<origin xyz="0.0 0.0 0.0"/>
+    	<parent link="base_footprint"/>
+    	<child link="base_link"/>
+ 	</joint>
+ 	<link name="base_footprint">
+ 	</link>
 	<!-- base of robot-->
 	<xacro:macro name="base_link">
@@ -172,3 +180,33 @@
 	<xacro:trans prefix="left_front"/>
 	<xacro:trans prefix="left_back"/>
+	<joint name="imu_joint" type="fixed">
+    	<axis xyz="0 0 0"/>
+    	<origin xyz="0.0 0.0 0.0"/>
+    	<parent link="base_link"/>
+    	<child link="imu_link"/>
+ 	</joint>
+ 	<link name="imu_link">
+ 		<inertial>
+ 			<mass value="0.001"/>
+ 			<origin rpy="0.0 0.0 0.0" xyz="0.0 0.0 0.0"/>
+ 			<inertia ixx="0.0001" ixy="0" ixz="0" iyy="0.000001" iyz="0" izz="0.0001"/>
+ 		</inertial>
+ 		<collision>
+ 			<origin rpy="0 0 0" xyz="0 0 0"/>
+ 			<geometry>
+ 				<box size=".001 .001 .001"/>
+ 			</geometry>
+ 		</collision>
+ 	</link>
+ 	<gazebo>
+ 		<plugin filename="libgazebo_ros_imu.so" name="imu_en_ros">
+ 			<alwaysOn>true</alwaysOn>
+ 			<updateRate>100.0</updateRate>
+ 			<bodyName>imu_link</bodyName>
+ 			<topicName>imu_data</topicName>
+ 			<gaussianNoise>2.89e-08</gaussianNoise>
+ 			<xyzOffset>0.0 0.0 0.0</xyzOffset>
+ 			<rpyOffset>0.0 0.0 0.0</rpyOffset>
+ 		</plugin>
+ 	</gazebo>
 </robot>
